Commit message: Adding differential drive control plugin for Gazebo

File: adns_robot_sim/models/urdf/adns_robot.urdf (robot description, URDF)
Before this commit: robot adns_robot, 8 links, 7 joints
Links:
- link base_link: mass 1 -> 20

Commit message: Basic differential drive control finished

File: adns_robot_sim/models/urdf/adns_robot.urdf (robot description, URDF)
Before this commit: robot adns_robot, 8 links, 7 joints
Links:
- link b_l_wheel: mass 1 -> 0.5
- link b_r_wheel: mass 1 -> 0.5
- link base_link: mass 20 -> 10
- link container: mass 1 -> 30
- link f_l_wheel: mass 1 -> 0.5
- link f_r_wheel: mass 1 -> 0.5

Commit message: Adding depth camera to Gazebo sim

File: adns_robot_sim/models/urdf/adns_robot.urdf (robot description, URDF)
Before this commit: robot adns_robot, 8 links, 7 joints
Links:
- removed link camera
- added link camera_link, mass 0.5; collision box size=0.012 0.139 0.026; visual box size=0.012 0.139 0.026
- link tilt_bracket: mass None -> 0.5; geometry collision box size=0.03 0.03 0.03; visual box size=0.03 0.03 0.03
Joints:
- joint pan_servo_joint: origin xyz=0 0 0.1397 -> xyz=0.1016 0 0.1397; type revolute -> fixed
- joint tilt_servo_joint: child camera -> camera_link; origin xyz=0 0 0.02 -> xyz=0 0 0.04; type revolute -> fixed

Commit message: Minor tweaks, adding aruco_detect node

File: adns_robot_sim/models/urdf/adns_robot.urdf (robot description, URDF)
Before this commit: robot adns_robot, 8 links, 7 joints
Links:
- link tilt_bracket: geometry collision box size=0.03 0.03 0.03; visual box size=0.012 0.03 0.03
Joints:
- joint pan_servo_joint: origin xyz=0.1016 0 0.1397 -> xyz=0.1524 0 0.1397
